File: PCB/Jarned V1.kicad_pcb (KiCad board)
At the start: 2 copper layers, 77 x 69.5 mm, 8 parts, among them J1 Conn_01x04, SW1 SW_Push, SW2 SW_Push, SW3 SW_Push, SW4 RotaryEncoder_Switch, SW5 SW_Push, SW6 SW_Push, U1 MOUDLE-SEEEDUINO-XIAO

Commit message: Updates KiCad skematics
Parts:
- moved J1 8.19 mm to (219.0, 78.9), turned to -90 degrees
Routing:
- net GND: track 198.6 -> 187.0 mm
- net /SDA: track 29.4 -> 18.5 mm
- net /SCL: track 39.8 -> 32.8 mm
- net /VVC: track 37.6 -> 38.8 mm
Other:
- board text added: "69.50"
- board text added: "70mm"
